File: MidtownDoorNumbers-LEDStrip.kicad_pcb (KiCad board)
At the start: 2 copper layers, 60 x 16 mm, 18 parts, among them J1 CONN_01X04, J2 CONN_01X04

Commit message: Generated Gerbers
Parts:
- added G***: LOGO, NilesLogos:HakcerLabHLogo-10mm, B.Cu at (118.9, 106.2)
- added REF***: OSHW-Symbol_8.9x8mm_SilkScreen, Symbols:OSHW-Symbol_8.9x8mm_SilkScreen, B.Cu at (129.8, 106.1)
- added nilesface: , NilesLogos:nilesface_smaller, B.Cu at (136.4, 110.0)
