File: MidtownDoorNumbers.kicad_pcb (KiCad board)
At the start: 2 copper layers, 60 x 45 mm, 17 parts, among them J1 CONN_01X02, J2 CONN_02X02, J3 CONN_01X04, J6 CONN_01X04, SW1 SW_DIP_x05, U1 LM7805CT, U2 NodeMCU_Amica_R2, U3 74AHC125, U4 74HC165

Commit message: Generated Gerbers
Parts:
- added G***: LOGO, NilesLogos:HakcerLabHLogo-10mm, B.Cu at (124.7, 68.9)
- added REF***: OSHW-Symbol_13.4x12mm_SilkScreen, Symbols:OSHW-Symbol_13.4x12mm_SilkScreen, B.Cu at (111.2, 69.3)
- added nilesface: , nilesface2:nilesface_smaller, F.Cu at (134.6, 93.0)
- added nilesface: , nilesface2:nilesface_smaller, B.Cu at (131.1, 73.2)
